File: PCB_Layouts/GigE_Module/GigE_Module.kicad_pcb (KiCad board)
At the start: 2 copper layers, 33.5 x 25.2 mm, 25 parts, among them J1 RJ45_LED, J2 Conn_01x10_Socket, J3 Conn_01x10_Socket, U4 ENC28J60x-SS, Y1 25MHz

Commit message: Updating USB and GigE files for PCB quotes
Parts:
- C1: footprint Capacitor_Tantalum_SMD:CP_EIA-1608-08_AVX-J -> Capacitor_SMD:CP_Elec_4x5.4; moved to F.Cu
- C10, C2, C3, C4, C5, C6, C7, C8: footprint Capacitor_Tantalum_SMD:CP_EIA-1608-08_AVX-J -> Capacitor_SMD:C_0603_1608Metric
- C9: value 0.01u -> 100nF; footprint Capacitor_Tantalum_SMD:CP_EIA-1608-08_AVX-J -> Capacitor_SMD:C_0603_1608Metric
- L1: footprint Inductor_SMD:L_0603_1608Metric -> Inductor_SMD:L_0201_0603Metric_Pad0.64x0.40mm_HandSolder
- Y1: footprint Crystal:Crystal_SMD_MicroCrystal_CC4V-T1A-2Pin_5.0x1.9mm -> Crystal:Crystal_SMD_MicroCrystal_CC8V-T1A-2Pin_2.0x1.2mm
- moved C1 11.8 mm to (139.2, 88.6)
- moved Y1 1.52 mm to (138.3, 86.2)
- moved L1 1.17 mm to (139.4, 99.1), turned to 180 degrees
- renumbered U4 to U1
Routing:
- net Net-(U1-VCAP): track 2.21 -> 9.99 mm, vias 0 -> 1
- net Net-(U1-OSC1): track 6.06 -> 10.7 mm
- net /GND: track 100.4 -> 104.1 mm
- net /VCC: track 98.2 -> 100.9 mm
- net Net-(C9-Pad1): track 15.8 -> 17.5 mm
