File: PCB_Layouts/GigE_Module/GigE_Module.kicad_sch (KiCad schematic)
At the start: 25 parts, among them J1 RJ45_LED, J2 Conn_01x10_Socket, J3 Conn_01x10_Socket, U4 ENC28J60x-SS, Y1 25MHz

Commit message: Updating USB and GigE files for PCB quotes
Parts:
- C1: footprint Capacitor_Tantalum_SMD:CP_EIA-1608-08_AVX-J -> Capacitor_SMD:CP_Elec_4x5.4
- C10, C2, C3, C4, C5, C6, C7, C8: footprint Capacitor_Tantalum_SMD:CP_EIA-1608-08_AVX-J -> Capacitor_SMD:C_0603_1608Metric
- C9: value 0.01u -> 100nF; footprint Capacitor_Tantalum_SMD:CP_EIA-1608-08_AVX-J -> Capacitor_SMD:C_0603_1608Metric
- L1: footprint Inductor_SMD:L_0603_1608Metric -> Inductor_SMD:L_0201_0603Metric_Pad0.64x0.40mm_HandSolder
- Y1: footprint Crystal:Crystal_SMD_MicroCrystal_CC4V-T1A-2Pin_5.0x1.9mm -> Crystal:Crystal_SMD_MicroCrystal_CC8V-T1A-2Pin_2.0x1.2mm
- renumbered U4 to U1
Changed lines of the file:
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@@
       (effects (font (size 1.27 1.27)) (justify left))
     )
-    (property "Footprint" "Capacitor_Tantalum_SMD:CP_EIA-1608-08_AVX-J" (at 94.9452 57.15 0)
+    (property "Footprint" "Capacitor_SMD:C_0603_1608Metric" (at 94.9452 57.15 0)
       (effects (font (size 1.27 1.27)) hide)
     )
@@
       (effects (font (size 1.27 1.27)) (justify left))
     )
-    (property "Footprint" "Capacitor_Tantalum_SMD:CP_EIA-1608-08_AVX-J" (at 182.5752 91.44 0)
+    (property "Footprint" "Capacitor_SMD:CP_Elec_4x5.4" (at 182.5752 91.44 0)
       (effects (font (size 1.27 1.27)) hide)
     )
@@
       (effects (font (size 1.27 1.27)) (justify left))
     )
-    (property "Footprint" "Capacitor_Tantalum_SMD:CP_EIA-1608-08_AVX-J" (at 233.3752 74.93 0)
+    (property "Footprint" "Capacitor_SMD:C_0603_1608Metric" (at 233.3752 74.93 0)
       (effects (font (size 1.27 1.27)) hide)
     )
@@
       (effects (font (size 1.27 1.27)) (justify left))
     )
-    (property "Footprint" "Capacitor_Tantalum_SMD:CP_EIA-1608-08_AVX-J" (at 107.6452 162.56 0)
+    (property "Footprint" "Capacitor_SMD:C_0603_1608Metric" (at 107.6452 162.56 0)
       (effects (font (size 1.27 1.27)) hide)
     )
@@
       (effects (font (size 1.27 1.27)))
     )
-    (property "Footprint" "Capacitor_Tantalum_SMD:CP_EIA-1608-08_AVX-J" (at 107.95 59.9948 0)
+    (property "Footprint" "Capacitor_SMD:C_0603_1608Metric" (at 107.95 59.9948 0)
       (effects (font (size 1.27 1.27)) hide)
     )
@@
       (effects (font (size 1.27 1.27)))
     )
-    (property "Footprint" "Capacitor_Tantalum_SMD:CP_EIA-1608-08_AVX-J" (at 107.95 80.3148 0)
+    (property "Footprint" "Capacitor_SMD:C_0603_1608Metric" (at 107.95 80.3148 0)
       (effects (font (size 1.27 1.27)) hide)
     )
@@
       (effects (font (size 1.27 1.27)) (justify left))
     )
-    (property "Footprint" "Crystal:Crystal_SMD_MicroCrystal_CC4V-T1A-2Pin_5.0x1.9mm" (at 114.3 71.12 0)
+    (property "Footprint" "Crystal:Crystal_SMD_MicroCrystal_CC8V-T1A-2Pin_2.0x1.2mm" (at 114.3 71.12 0)
       (effects (font (size 1.27 1.27)) hide)
     )
@@
       (effects (font (size 1.27 1.27)) (justify left))
     )
-    (property "Footprint" "Capacitor_Tantalum_SMD:CP_EIA-1608-08_AVX-J" (at 243.5352 74.93 0)
+    (property "Footprint" "Capacitor_SMD:C_0603_1608Metric" (at 243.5352 74.93 0)
       (effects (font (size 1.27 1.27)) hide)
     )
@@
       (effects (font (size 1.27 1.27)) (justify left))
     )
-    (property "Footprint" "Capacitor_Tantalum_SMD:CP_EIA-1608-08_AVX-J" (at 223.2152 74.93 0)
+    (property "Footprint" "Capacitor_SMD:C_0603_1608Metric" (at 223.2152 74.93 0)
       (effects (font (size 1.27 1.27)) hide)
     )
@@
   (symbol (lib_id "Interface_Ethernet:ENC28J60x-SS") (at 156.21 60.96 0) (unit 1)
     (in_bom yes) (on_board yes) (dnp no) (fields_autoplaced)
-    (property "Reference" "U4" (at 160.9441 33.02 0)
+    (property "Reference" "U1" (at 160.9441 33.02 0)
       (effects (font (size 1.27 1.27)) (justify left))
     )
@@
       (project "GigE_Module"
         (path "/670fdc0c-f766-4a3d-acb5-c6529564e189"
-          (reference "U4") (unit 1)
+          (reference "U1") (unit 1)
         )
       )
@@
       (effects (font (size 1.27 1.27)))
     )
-    (property "Value" "0.01u" (at 142.24 110.49 90)
-      (effects (font (size 1.27 1.27)))
-    )
-    (property "Footprint" "Capacitor_Tantalum_SMD:CP_EIA-1608-08_AVX-J" (at 146.05 114.6048 0)
+    (property "Value" "100nF" (at 142.24 110.49 90)
+      (effects (font (size 1.27 1.27)))
+    )
+    (property "Footprint" "Capacitor_SMD:C_0603_1608Metric" (at 146.05 114.6048 0)
       (effects (font (size 1.27 1.27)) hide)
     )
@@
       (effects (font (size 1.27 1.27)) (justify left))
     )
-    (property "Footprint" "Capacitor_Tantalum_SMD:CP_EIA-1608-08_AVX-J" (at 213.0552 74.93 0)
+    (property "Footprint" "Capacitor_SMD:C_0603_1608Metric" (at 213.0552 74.93 0)
       (effects (font (size 1.27 1.27)) hide)
     )
@@
       (effects (font (size 1.27 1.27)))
     )
-    (property "Footprint" "Inductor_SMD:L_0603_1608Metric" (at 116.84 115.57 0)
-      (effects (font (size 1.27 1.27)) hide)
-    )
+    (property "Footprint" "Inductor_SMD:L_0201_0603Metric_Pad0.64x0.40mm_HandSolder" (at 116.84 115.57 0)
+      (effects (font (size 1.27 1.27)) hide)
+    )
