File: PCB_Layouts/FPV_3-Pin_Module/FPV_3-Pin_Module.kicad_sch (KiCad schematic)
At the start: 3 parts, among them J1 Conn_01x03_Socket, J2 Conn_01x10_Socket, J3 Conn_01x10_Socket

Commit message: Adding FPV 3 Pin quote
Parts:
- J1: footprint Connector_JST:JST_PH_B3B-PH-K_1x03_P2.00mm_Vertical -> Connector_JST:JST_XH_B3B-XH-A_1x03_P2.50mm_Vertical
Changed lines of the file:
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@@
       (effects (font (size 1.27 1.27)))
     )
-    (property "Footprint" "Connector_JST:JST_PH_B3B-PH-K_1x03_P2.00mm_Vertical" (at 142.24 93.98 0)
+    (property "Footprint" "Connector_JST:JST_XH_B3B-XH-A_1x03_P2.50mm_Vertical" (at 142.24 93.98 0)
       (effects (font (size 1.27 1.27)) hide)
     )
